Commit message: refactor(xacro): cleaned agri_rover.xacro for better readability

File: model/agri_rover.xacro (robot description, xacro)
@@ -8,9 +8,10 @@
     <color rgba="1 0 0 1"/>
   </material>
+<!-- CHASSIS -->
   <link name= "base_footprint"></link>
   <link name="chassis">
     <visual>
       <origin
-        xyz="-0.0325699147746112 -0.0148144596659951 0.0176361848244046"
+        xyz="0 0 0.01"
         rpy="0 0 0" />
       <geometry>
@@ -24,21 +25,12 @@
       </material>
     </visual>
-    <inertial>
+    <xacro:inertial_box mass = "39.7761394814532" x = "1.202" y="0.674" z="0.650">
       <origin
-        xyz="-0.0325699147746112 -0.0148144596659951 0.0176361848244046"
+        xyz="0 0 0.01"
         rpy="0 0 0" />
-      <mass
-        value="39.7761394814532" />
-      <inertia
-        ixx="0.35694476106406"
-        ixy="-1.08000535961728E-05"
-        ixz="0.00834860225034306"
-        iyy="0.287498385304558"
-        iyz="-0.00209844360915769"
-        izz="0.477878098599329" />
-    </inertial>
+    </xacro:inertial_box>
     <collision>
       <origin
-        xyz="-0.0325699147746112 -0.0148144596659951 0.0176361848244046"
+        xyz="0 0 0.01"
         rpy="0 0 0" />
       <geometry>
@@ -49,9 +41,9 @@
   </link>
   <joint name="chassis_joint" type="fixed">
-    <origin xyz="0 0 0.57" rpy="0 0 0" />
+    <origin xyz="0 0 0.56" rpy="0 0 0" />
     <parent link="base_footprint" />
     <child link="chassis" />
   </joint>
-<!-- FRONT LEFT WHEEL-->
+<!-- FRONT LEFT WHEEL -->
 <joint name="fl_wheel_joint" type="continuous">
   <parent link="chassis"/>
@@ -76,14 +68,9 @@
     </geometry>
   </collision>
-<inertial>
-  <mass value="1.0"/>
-  <origin xyz="0 0 0" rpy="0 0 0"/>
-  <inertia
-    ixx="0.01" ixy="0.0" ixz="0.0"
-    iyy="0.01" iyz="0.0"
-    izz="0.01"/>
-</inertial>
-</link>
-<!-- FRONT RIGHT WHEEL-->
+  <xacro:inertial_cylinder mass="2.0" length="0.04" radius="0.1">
+    <origin xyz="0 0 0" rpy="0 0 0"/>
+  </xacro:inertial_cylinder>
+</link>
+<!-- FRONT RIGHT WHEEL -->
 <joint name="fr_wheel_joint" type="continuous">
   <parent link="chassis"/>
@@ -108,14 +95,9 @@
     </geometry>
   </collision>
-<inertial>
-  <mass value="1.0"/>
-  <origin xyz="0 0 0" rpy="0 0 0"/>
-  <inertia
-    ixx="0.01" ixy="0.0" ixz="0.0"
-    iyy="0.01" iyz="0.0"
-    izz="0.01"/>
-</inertial>
-</link>
-<!-- MIDDLE LEFT WHEEL-->
+  <xacro:inertial_cylinder mass="2.0" length="0.04" radius="0.1">
+    <origin xyz="0 0 0" rpy="0 0 0"/>
+  </xacro:inertial_cylinder>
+</link>
+<!-- MIDDLE LEFT WHEEL -->
 <joint name="ml_wheel_joint" type="continuous">
   <parent link="chassis"/>
@@ -140,14 +122,9 @@
     </geometry>
   </collision>
-<inertial>
-  <mass value="1.0"/>
-  <origin xyz="0 0 0" rpy="0 0 0"/>
-  <inertia
-    ixx="0.01" ixy="0.0" ixz="0.0"
-    iyy="0.01" iyz="0.0"
-    izz="0.01"/>
-</inertial>
-</link>
-<!-- MIDDLE RIGHT WHEEL-->
+  <xacro:inertial_cylinder mass="2.0" length="0.04" radius="0.1">
+    <origin xyz="0 0 0" rpy="0 0 0"/>
+  </xacro:inertial_cylinder>
+</link>
+<!-- MIDDLE RIGHT WHEEL -->
 <joint name="mr_wheel_joint" type="continuous">
   <parent link="chassis"/>
@@ -172,14 +149,9 @@
     </geometry>
   </collision>
-<inertial>
-  <mass value="1.0"/>
-  <origin xyz="0 0 0" rpy="0 0 0"/>
-  <inertia
-    ixx="0.01" ixy="0.0" ixz="0.0"
-    iyy="0.01" iyz="0.0"
-    izz="0.01"/>
-</inertial>
-</link>
-<!-- REAR LEFT WHEEL-->
+  <xacro:inertial_cylinder mass="2.0" length="0.04" radius="0.1">
+    <origin xyz="0 0 0" rpy="0 0 0"/>
+  </xacro:inertial_cylinder>
+</link>
+<!-- REAR LEFT WHEEL -->
 <joint name="rl_wheel_joint" type="continuous">
   <parent link="chassis"/>
@@ -204,14 +176,9 @@
     </geometry>
   </collision>
-<inertial>
-  <mass value="1.0"/>
-  <origin xyz="0 0 0" rpy="0 0 0"/>
-  <inertia
-    ixx="0.01" ixy="0.0" ixz="0.0"
-    iyy="0.01" iyz="0.0"
-    izz="0.01"/>
-</inertial>
-</link>
-<!-- REAR RIGHT WHEEL-->
+  <xacro:inertial_cylinder mass="2.0" length="0.04" radius="0.1">
+    <origin xyz="0 0 0" rpy="0 0 0"/>
+  </xacro:inertial_cylinder>
+</link>
+<!-- REAR RIGHT WHEEL -->
 <joint name="rr_wheel_joint" type="continuous">
   <parent link="chassis"/>
@@ -236,12 +203,7 @@
     </geometry>
   </collision>
-<inertial>
-  <mass value="1.0"/>
-  <origin xyz="0 0 0" rpy="0 0 0"/>
-  <inertia
-    ixx="0.01" ixy="0.0" ixz="0.0"
-    iyy="0.01" iyz="0.0"
-    izz="0.01"/>
-</inertial>
+  <xacro:inertial_cylinder mass="2.0" length="0.04" radius="0.1">
+    <origin xyz="0 0 0" rpy="0 0 0"/>
+  </xacro:inertial_cylinder>
 </link>
 </robot>
